File: Frontend/Frontend.kicad_sch (KiCad schematic)
At the start: 0 parts

Commit message: add libraries and make some symbols/footprints
Parts:
- added PLL1: MAX2871ETJ_T, Package_DFN_QFN:TQFN-32-1EP_5x5mm_P0.5mm_EP3.1x3.1mm_ThermalVias, symbol cwradar:MAX2871ETJ_T
Connections:
- new net GND: PLL1.11 (GND_RF), PLL1.18 (GND_VCO), PLL1.21 (GND_TUNE), PLL1.27 (GND_DIG), PLL1.31 (GND_SD), PLL1.33 (EP), PLL1.8 (GND_CP), PLL1.9 (GND_PLL)

Commit message: seperate PCB into hierarchical sheets, start on MAX2871 pinout
Parts:
- removed PLL1: MAX2871ETJ_T, Package_DFN_QFN:TQFN-32-1EP_5x5mm_P0.5mm_EP3.1x3.1mm_ThermalVias, symbol cwradar:MAX2871ETJ_T
Other:
- added sheet ADC (adc.kicad_sch)
- added sheet Baseband_I (baseband.kicad_sch)
- added sheet Baseband_Q (baseband.kicad_sch)
- added sheet Battery_Charger (battery_charger.kicad_sch)
- added sheet MCU (mcu.kicad_sch)
- added sheet Mechanical (mechanical.kicad_sch)
- added sheet Receiver (receiver.kicad_sch)
- added sheet Regulators (regulators.kicad_sch)
- added sheet Synthesizer (synthesizer.kicad_sch)
- added sheet User_IO (user_io.kicad_sch)
- company: (none) -> Senior Design
- title: (none) -> CW Radar Main Board
