File: Frontend/mechanical.kicad_sch (KiCad schematic)
At the start: 0 parts

Commit message: floorplan PCB some, draw out I/Q and VCO schematics
Parts:
- added MH1101, MH1102, MH1103, MH1104: M3, MountingHole:MountingHole_3.2mm_M3_Pad_Via, symbol Mechanical:MountingHole_Pad
Connections:
- new net GND: MH1101.1, MH1102.1, MH1103.1, MH1104.1
Other:
- note added: "M3 plated holes tied to GND, one per corner."
- note added: "MOUNTING"
