File: Frontend/synthesizer.kicad_sch (KiCad schematic)
At the start: 45 parts, among them J601 TX, J602 MON

Commit message: floorplan PCB some, draw out I/Q and VCO schematics
Parts:
- removed C623: 100n, Capacitor_SMD:C_0402_1005Metric, symbol cwradar:100n
- added C623: 100n, cwradar:C_Panasonic_ECHU_E2, symbol cwradar:100n_PPS
- added C625, C628: 1u, Capacitor_SMD:C_0402_1005Metric, symbol cwradar:1u
- added C626, C627: TBD, Capacitor_SMD:C_0402_1005Metric, symbol Device:C
- added R618: 0R, Resistor_SMD:R_0603_1608Metric, symbol cwradar:0R
- added R619: 100k, Resistor_SMD:R_0402_1005Metric, symbol cwradar:100k
- added TP602: TUNE, TestPoint:TestPoint_Pad_D1.0mm, symbol Connector:TestPoint
- added Y601: 25 MHz TCXO ±2.5 ppm clipped-sine — PART TBD, symbol cwradar:TCXO_2520
- J601: value TX -> TX SMA; footprint (none) -> Connector_Coaxial:SMA_Molex_73251-1153_EdgeMount_Horizontal; Manufacturer (none) -> Molex; Mfg Part # (none) -> 73251-1153
- J602: value MON -> MON SMA; footprint Connector_Coaxial:U.FL_Hirose_U.FL-R-SMT-1_Vertical -> Connector_Coaxial:SMA_Molex_73251-1153_EdgeMount_Horizontal; Manufacturer (none) -> Molex; Mfg Part # (none) -> 73251-1153
- PLL601: footprint Package_DFN_QFN:TQFN-32-1EP_5x5mm_P0.5mm_EP3.1x3.1mm_ThermalVias -> cwradar:TQFN-32-1EP_5x5mm_P0.5mm_EP3.1x3.1mm_ThermalVias0.3
- TP601: now left out of the parts list
Connections:
- net +3V3_SYN: now also R618.1
- net +3V3_SYN_DIG: now also C628.1
- net +3V3_SYN_REF: now also Y601.4 (Vcc)
- net +3V3_SYN_RF: now also C626.1, C627.1; no longer C613.1, PLL601.17 (VCC_VCO)
- net GND: now also C623.2, C625.2, C626.2, C627.2, C628.2, Y601.2 (GND)
- net LF_C2: now also C623.1
- net REF_25M: now also Y601.3 (OUT)
- net TUNE: now also R619.1
- new net +3V3_SYN_VCO: C613.1, C625.1, PLL601.17 (VCC_VCO), R618.2
- new net TUNE_TP: R619.2, TP602.1
- no-connect marks 1 -> 2
Other:
- note added: "Place at R611/R613 supply end"
- note added: "Place at R614/R615 supply end"
